File: fox50.kicad_sch (KiCad schematic)
At the start: 0 parts

Commit message: simbolos
Parts:
- added D? (x56): D_Small, symbol res:D_Small
- added MX? (x56): MX-NoLED, symbol mx:MX-NoLED
Connections:
- new net: D?.2 (A), MX?.2 (ROW) (x56)
