File: fox50.kicad_sch (KiCad schematic)
At the start: 112 parts

Commit message: conexiones del eschema
Parts:
- removed D? (x8): D_Small, symbol res:D_Small
- removed MX? (x8): MX-NoLED, symbol mx:MX-NoLED
Connections:
- net at D?.1 (K): now also D?.1 (K), D?.1 (K), D?.1 (K), D?.1 (K), D?.1 (K), D?.1 (K), D?.1 (K), D?.1 (K), D?.1 (K), D?.1 (K), D?.1 (K), D?.1 (K) (x2)
- net at MX?.1 (COL): now also MX?.1 (COL), MX?.1 (COL), MX?.1 (COL) (x8)
- net at MX?.1 (COL): now also MX?.1 (COL), MX?.1 (COL) (x5)
- net at D?.1 (K): now also D?.1 (K), D?.1 (K), D?.1 (K), D?.1 (K), D?.1 (K), D?.1 (K), D?.1 (K)
- net at D?.1 (K): now also D?.1 (K), D?.1 (K), D?.1 (K), D?.1 (K), D?.1 (K)

Commit message: cols and rows
Parts:
- added U1: ProMicro, keyboard_parts:Pro_Micro, symbol cpu:ProMicro
- D1, D10, D11, D12, D13, D14, D15, D16, D17, D18, D19, D2, D20, D21, D22, D23, D24, D25, D26, D27, D28, D29, D3, D30, D31, D32, D33, D34, D35, D36, D37, D38, D39, D4, D40, D41, D42, D43, D44, D45, D46, D47, D5, D6, D7, D8, D9: renamed from D?; footprint (none) -> keyboard_parts:D_1206
- D48: renamed from D?; footprint (none) -> Button_Switch_Keyboard:SW_Cherry_MX_1.00u_PCB
- MX1, MX10, MX11, MX12, MX13, MX14, MX15, MX16, MX17, MX18, MX19, MX2, MX20, MX21, MX22, MX23, MX24, MX25, MX26, MX27, MX28, MX29, MX3, MX30, MX31, MX32, MX33, MX34, MX35, MX36, MX37, MX38, MX39, MX4, MX40, MX41, MX42, MX43, MX44, MX45, MX46, MX47, MX48, MX5, MX6, MX7, MX8, MX9: renamed from MX?; footprint (none) -> Button_Switch_Keyboard:SW_Cherry_MX_1.00u_PCB
Connections:
- net row2: now reaches D11.1 (K), D15.1 (K), D19.1 (K), D23.1 (K), D27.1 (K), D3.1 (K), D31.1 (K), D35.1 (K), D38.1 (K), D41.1 (K), D44.1 (K), D47.1 (K), D7.1 (K)
- net row0: now reaches D33.1 (K)
- net row0: now also D1.1 (K), D13.1 (K), D17.1 (K), D21.1 (K), D25.1 (K), D29.1 (K), D36.1 (K), D39.1 (K), D42.1 (K), D45.1 (K), D48.1 (K), D5.1 (K), D9.1 (K)
- net col1: now reaches MX13.1 (COL), MX14.1 (COL), MX15.1 (COL), MX16.1 (COL)
- net col1: now also MX1.1 (COL), MX10.1 (COL), MX11.1 (COL), MX12.1 (COL), MX17.1 (COL), MX18.1 (COL), MX19.1 (COL), MX2.1 (COL), MX20.1 (COL), MX21.1 (COL), MX22.1 (COL), MX23.1 (COL), MX24.1 (COL), MX25.1 (COL), MX26.1 (COL), MX27.1 (COL), MX28.1 (COL), MX29.1 (COL), MX3.1 (COL), MX30.1 (COL), MX31.1 (COL), MX32.1 (COL), MX33.1 (COL), MX34.1 (COL), MX35.1 (COL), MX36.1 (COL), MX37.1 (COL), MX38.1 (COL), MX39.1 (COL), MX4.1 (COL), MX40.1 (COL), MX41.1 (COL), MX42.1 (COL), MX43.1 (COL), MX44.1 (COL), MX45.1 (COL), MX46.1 (COL), MX47.1 (COL), MX48.1 (COL), MX5.1 (COL), MX6.1 (COL), MX7.1 (COL), MX8.1 (COL), MX9.1 (COL)
- net row3: now reaches D12.1 (K), D16.1 (K), D20.1 (K), D24.1 (K), D28.1 (K), D32.1 (K), D4.1 (K), D8.1 (K)

Commit message: fix nets
Connections:
- net col1: no longer MX10.1 (COL), MX11.1 (COL), MX12.1 (COL), MX13.1 (COL), MX14.1 (COL), MX15.1 (COL), MX16.1 (COL), MX17.1 (COL), MX18.1 (COL), MX19.1 (COL), MX20.1 (COL), MX21.1 (COL), MX22.1 (COL), MX23.1 (COL), MX24.1 (COL), MX25.1 (COL), MX26.1 (COL), MX27.1 (COL), MX28.1 (COL), MX29.1 (COL), MX30.1 (COL), MX31.1 (COL), MX32.1 (COL), MX33.1 (COL), MX34.1 (COL), MX35.1 (COL), MX36.1 (COL), MX37.1 (COL), MX38.1 (COL), MX39.1 (COL), MX40.1 (COL), MX41.1 (COL), MX42.1 (COL), MX43.1 (COL), MX44.1 (COL), MX45.1 (COL), MX46.1 (COL), MX47.1 (COL), MX48.1 (COL), MX5.1 (COL), MX6.1 (COL), MX7.1 (COL), MX8.1 (COL), MX9.1 (COL)
- new net col10: MX36.1 (COL), MX37.1 (COL), MX38.1 (COL)
- new net col11: MX24.1 (COL), MX39.1 (COL), MX40.1 (COL), MX41.1 (COL)
- new net col12: MX28.1 (COL), MX42.1 (COL), MX43.1 (COL), MX44.1 (COL)
- new net col13: MX32.1 (COL), MX45.1 (COL), MX46.1 (COL), MX47.1 (COL)
- new net col14: MX48.1 (COL)
- new net col2: MX5.1 (COL), MX6.1 (COL), MX7.1 (COL), MX8.1 (COL)
- new net col3: MX10.1 (COL), MX11.1 (COL), MX12.1 (COL), MX9.1 (COL)
- new net col4: MX13.1 (COL), MX14.1 (COL), MX15.1 (COL), MX16.1 (COL)
- new net col5: MX17.1 (COL), MX18.1 (COL), MX19.1 (COL), MX20.1 (COL)
- new net col6: MX21.1 (COL), MX22.1 (COL), MX23.1 (COL)
- new net col7: MX25.1 (COL), MX26.1 (COL), MX27.1 (COL)
- new net col8: MX29.1 (COL), MX30.1 (COL), MX31.1 (COL)
- new net col9: MX33.1 (COL), MX34.1 (COL), MX35.1 (COL)
Other:
- moved on the sheet: D24, D28, D32, MX24, MX28, MX32
