File: fox50.kicad_pcb (KiCad board)
At the start: 2 copper layers, 97 parts, among them U1 ProMicro

Commit message: nets done 2
Connections:
- MX10 pad 1: col1 -> col3
- MX11 pad 1: col1 -> col3
- MX12 pad 1: col1 -> col3
- MX13 pad 1: col1 -> col4
- MX14 pad 1: col1 -> col4
- MX15 pad 1: col1 -> col4
- MX16 pad 1: col1 -> col4
- MX17 pad 1: col1 -> col5
- MX18 pad 1: col1 -> col5
- MX19 pad 1: col1 -> col5
- MX20 pad 1: col1 -> col5
- MX21 pad 1: col1 -> col6
- MX22 pad 1: col1 -> col6
- MX23 pad 1: col1 -> col6
- MX24 pad 1: col1 -> col11
- MX25 pad 1: col1 -> col7
- MX26 pad 1: col1 -> col7
- MX27 pad 1: col1 -> col7
- MX28 pad 1: col1 -> col12
- MX29 pad 1: col1 -> col8
- MX30 pad 1: col1 -> col8
- MX31 pad 1: col1 -> col8
- MX32 pad 1: col1 -> col13
- MX33 pad 1: col1 -> col9
- MX34 pad 1: col1 -> col9
- MX35 pad 1: col1 -> col9
- MX36 pad 1: col1 -> col10
- MX37 pad 1: col1 -> col10
- MX38 pad 1: col1 -> col10
- MX39 pad 1: col1 -> col11
- MX40 pad 1: col1 -> col11
- MX41 pad 1: col1 -> col11
- MX42 pad 1: col1 -> col12
- MX43 pad 1: col1 -> col12
- MX44 pad 1: col1 -> col12
- MX45 pad 1: col1 -> col13
- MX46 pad 1: col1 -> col13
- MX47 pad 1: col1 -> col13
- MX48 pad 1: col1 -> col14
- MX5 pad 1: col1 -> col2
- MX6 pad 1: col1 -> col2
- MX7 pad 1: col1 -> col2
- MX8 pad 1: col1 -> col2
- MX9 pad 1: col1 -> col3

Commit message: red net done
Routing:
- net col5: track 0.00 -> 93.2 mm
- net col3: track 0.00 -> 75.3 mm
- net col4: track 0.00 -> 72.1 mm
- net col13: track 0.00 -> 70.8 mm
- net col12: track 0.00 -> 67.0 mm
- net col11: track 0.00 -> 66.0 mm
- net col2: track 0.00 -> 64.1 mm
- net col1: track 0.00 -> 57.1 mm
- net col7: track 0.00 -> 44.0 mm
- net col9: track 0.00 -> 44.0 mm
- net col8: track 0.00 -> 44.0 mm
- net col6: track 0.00 -> 44.0 mm
- net col10: track 0.00 -> 44.0 mm
Changed lines of the file:
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@@
     (thickness 1.6)
     (drawings 0)
-    (tracks 0)
+    (tracks 78)
     (modules 97)
     (nets 91)
@@
     )
   )
+  (segment (start 137.4775 39.37) (end 137.4775 48.895) (width 0.25) (layer "F.Cu") (net 82))
+  (segment (start 137.4775 48.895) (end 147.0025 58.42) (width 0.25) (layer "F.Cu") (net 82))
+  (segment (start 132.715 20.32) (end 132.715 34.6075) (width 0.25) (layer "F.Cu") (net 82))
+  (segment (start 132.715 34.6075) (end 137.4775 39.37) (width 0.25) (layer "F.Cu") (net 82))
+  (segment (start 156.5275 39.37) (end 156.5275 48.895) (width 0.25) (layer "F.Cu") (net 83))
+  (segment (start 156.5275 48.895) (end 166.0525 58.42) (width 0.25) (layer "F.Cu") (net 83))
+  (segment (start 151.765 20.32) (end 151.765 34.6075) (width 0.25) (layer "F.Cu") (net 83))
+  (segment (start 151.765 34.6075) (end 156.5275 39.37) (width 0.25) (layer "F.Cu") (net 83))
+  (segment (start 175.5775 39.37) (end 175.5775 48.895) (width 0.25) (layer "F.Cu") (net 84))
+  (segment (start 175.5775 48.895) (end 185.1025 58.42) (width 0.25) (layer "F.Cu") (net 84))
+  (segment (start 170.815 20.32) (end 170.815 34.6075) (width 0.25) (layer "F.Cu") (net 84))
+  (segment (start 170.815 34.6075) (end 175.5775 39.37) (width 0.25) (layer "F.Cu") (net 84))
+  (segment (start 194.6275 39.37) (end 194.6275 48.895) (width 0.25) (layer "F.Cu") (net 85))
+  (segment (start 194.6275 48.895) (end 204.1525 58.42) (width 0.25) (layer "F.Cu") (net 85))
+  (segment (start 189.865 20.32) (end 189.865 34.6075) (width 0.25) (layer "F.Cu") (net 85))
+  (segment (start 189.865 34.6075) (end 194.6275 39.37) (width 0.25) (layer "F.Cu") (net 85))
+  (segment (start 213.6775 39.37) (end 213.6775 48.895) (width 0.25) (layer "F.Cu") (net 86))
+  (segment (start 213.6775 48.895) (end 223.2025 58.42) (width 0.25) (layer "F.Cu") (net 86))
+  (segment (start 208.915 20.32) (end 208.915 34.6075) (width 0.25) (layer "F.Cu") (net 86))
+  (segment (start 208.915 34.6075) (end 213.6775 39.37) (width 0.25) (layer "F.Cu") (net 86))
+  (segment (start 242.2525 58.42) (end 242.2525 70.32625) (width 0.25) (layer "F.Cu") (net 87))
+  (segment (start 242.2525 70.32625) (end 249.39625 77.47) (width 0.25) (layer "F.Cu") (net 87))
+  (segment (start 232.7275 39.37) (end 232.7275 48.895) (width 0.25) (layer "F.Cu") (net 87))
+  (segment (start 232.7275 48.895) (end 242.2525 58.42) (width 0.25) (layer "F.Cu") (net 87))
+  (segment (start 227.965 20.32) (end 227.965 34.6075) (width 0.25) (layer "F.Cu") (net 87))
+  (segment (start 227.965 34.6075) (end 232.7275 39.37) (width 0.25) (layer "F.Cu") (net 87))
+  (segment (start 261.3025 58.42) (end 261.3025 67.945) (width 0.25) (layer "F.Cu") (net 88))
+  (segment (start 261.3025 67.945) (end 270.8275 77.47) (width 0.25) (layer "F.Cu") (net 88))
+  (segment (start 251.7775 39.37) (end 251.7775 48.895) (width 0.25) (layer "F.Cu") (net 88))
+  (segment (start 251.7775 48.895) (end 261.3025 58.42) (width 0.25) (layer "F.Cu") (net 88))
+  (segment (start 247.015 20.32) (end 247.015 34.6075) (width 0.25) (layer "F.Cu") (net 88))
+  (segment (start 247.015 34.6075) (end 251.7775 39.37) (width 0.25) (layer "F.Cu") (net 88))
+  (segment (start 287.49625 58.42) (end 287.49625 72.7075) (width 0.25) (layer "F.Cu") (net 89))
+  (segment (start 287.49625 72.7075) (end 292.25875 77.47) (width 0.25) (layer "F.Cu") (net 89))
+  (segment (start 282.73375 39.37) (end 282.73375 53.6575) (width 0.25) (layer "F.Cu") (net 89))
+  (segment (start 282.73375 53.6575) (end 287.49625 58.42) (width 0.25) (layer "F.Cu") (net 89))
+  (segment (start 266.065 27.465) (end 274.35 35.75) (width 0.25) (layer "F.Cu") (net 89))
+  (segment (start 274.35 35.75) (end 279.11375 35.75) (width 0.25) (layer "F.Cu") (net 89))
+  (segment (start 266.065 20.32) (end 266.065 27.465) (width 0.25) (layer "F.Cu") (net 89))
+  (segment (start 279.11375 35.75) (end 282.73375 39.37) (width 0.25) (layer "F.Cu") (net 89))
+  (segment (start 128.5 62.8) (end 128.5 68.5) (width 0.25) (layer "F.Cu") (net 81))
+  (segment (start 127.9525 58.5025) (end 128.5 59.05) (width 0.25) (layer "F.Cu") (net 81))
+  (segment (start 127.9525 58.42) (end 127.9525 58.5025) (width 0.25) (layer "F.Cu") (net 81))
+  (segment (start 135 75) (end 137.95 75) (width 0.25) (layer "F.Cu") (net 81))
+  (segment (start 128.5 59.05) (end 128.5 62.8) (width 0.25) (layer "F.Cu") (net 81))
+  (segment (start 128.5 68.5) (end 135 75) (width 0.25) (layer "F.Cu") (net 81))
+  (segment (start 137.95 75) (end 161.20125 75) (width 0.25) (layer "F.Cu") (net 81))
+  (segment (start 161.20125 75) (end 163.67125 77.47) (width 0.25) (layer "F.Cu") (net 81))
+  (segment (start 118.4275 39.37) (end 118.4275 48.895) (width 0.25) (layer "F.Cu") (net 81))
+  (segment (start 118.4275 48.895) (end 127.9525 58.42) (width 0.25) (layer "F.Cu") (net 81))
+  (segment (start 113.665 20.32) (end 113.665 34.6075) (width 0.25) (layer "F.Cu") (net 81))
+  (segment (start 113.665 34.6075) (end 118.4275 39.37) (width 0.25) (layer "F.Cu") (net 81))
+  (segment (start 108.9025 58.42) (end 108.9025 64.401002) (width 0.25) (layer "F.Cu") (net 80))
+  (segment (start 108.9025 64.401002) (end 95.833502 77.47) (width 0.25) (layer "F.Cu") (net 80))
+  (segment (start 95.833502 77.47) (end 92.23375 77.47) (width 0.25) (layer "F.Cu") (net 80))
+  (segment (start 99.3775 39.37) (end 99.3775 48.895) (width 0.25) (layer "F.Cu") (net 80))
+  (segment (start 99.3775 48.895) (end 108.9025 58.42) (width 0.25) (layer "F.Cu") (net 80))
+  (segment (start 94.615 20.32) (end 94.615 34.6075) (width 0.25) (layer "F.Cu") (net 80))
+  (segment (start 94.615 34.6075) (end 99.3775 39.37) (width 0.25) (layer "F.Cu") (net 80))
+  (segment (start 89.8525 58.5525) (end 90.5 59.2) (width 0.25) (layer "F.Cu") (net 79))
+  (segment (start 89.8525 58.42) (end 89.8525 58.5525) (width 0.25) (layer "F.Cu") (net 79))
+  (segment (start 90.5 59.2) (end 90.5 64.3) (width 0.25) (layer "F.Cu") (net 79))
+  (segment (start 90.5 64.3) (end 80.8 74) (width 0.25) (layer "F.Cu") (net 79))
+  (segment (start 80.8 74) (end 74.2725 74) (width 0.25) (layer "F.Cu") (net 79))
+  (segment (start 74.2725 74) (end 70.8025 77.47) (width 0.25) (layer "F.Cu") (net 79))
+  (segment (start 80.3275 39.37) (end 80.3275 48.895) (width 0.25) (layer "F.Cu") (net 79))
+  (segment (start 80.3275 48.895) (end 89.8525 58.42) (width 0.25) (layer "F.Cu") (net 79))
+  (segment (start 75.565 20.32) (end 75.565 34.6075) (width 0.25) (layer "F.Cu") (net 79))
+  (segment (start 75.565 34.6075) (end 80.3275 39.37) (width 0.25) (layer "F.Cu") (net 79))
+  (segment (start 58.89625 58.42) (end 58.89625 67.945) (width 0.25) (layer "F.Cu") (net 78))
+  (segment (start 58.89625 67.945) (end 49.37125 77.47) (width 0.25) (layer "F.Cu") (net 78))
+  (segment (start 54.13375 39.37) (end 54.13375 53.6575) (width 0.25) (layer "F.Cu") (net 78))
+  (segment (start 54.13375 53.6575) (end 58.89625 58.42) (width 0.25) (layer "F.Cu") (net 78))
+  (segment (start 51.7525 20.32) (end 51.7525 36.98875) (width 0.25) (layer "F.Cu") (net 78))
+  (segment (start 51.7525 36.98875) (end 54.13375 39.37) (width 0.25) (layer "F.Cu") (net 78))
+  (segment (start 27.94 58.42) (end 27.94 77.47) (width 0.25) (layer "F.Cu") (net 53))
+  (segment (start 27.94 39.37) (end 27.94 58.42) (width 0.25) (layer "F.Cu") (net 53))
+  (segment (start 27.94 20.32) (end 27.94 39.37) (width 0.25) (layer "F.Cu") (net 53))
 )

Commit message: border done
Other:
- board outline added: 287.5 x 78 mm
Changed lines of the file:
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@@
   (general
     (thickness 1.6)
-    (drawings 0)
+    (drawings 8)
     (tracks 78)
     (modules 97)
@@
     )
   )
+  (gr_arc (start 302 15.5) (end 302.5 15.5) (angle -90) (layer "Edge.Cuts") (width 0.1))
+  (gr_arc (start 302 92.5) (end 302 93) (angle -90) (layer "Edge.Cuts") (width 0.1))
+  (gr_arc (start 15.5 92.5) (end 15 92.5) (angle -90) (layer "Edge.Cuts") (width 0.1))
+  (gr_arc (start 15.5 15.5) (end 15.5 15) (angle -90) (layer "Edge.Cuts") (width 0.1))
+  (gr_line (start 302 15) (end 15.5 15) (layer "Edge.Cuts") (width 0.1))
+  (gr_line (start 302.5 92.5) (end 302.5 15.5) (layer "Edge.Cuts") (width 0.1))
+  (gr_line (start 15.5 93) (end 302 93) (layer "Edge.Cuts") (width 0.1))
+  (gr_line (start 15 15.5) (end 15 92.5) (layer "Edge.Cuts") (width 0.1))
   (segment (start 137.4775 39.37) (end 137.4775 48.895) (width 0.25) (layer "F.Cu") (net 82))
   (segment (start 137.4775 48.895) (end 147.0025 58.42) (width 0.25) (layer "F.Cu") (net 82))

Commit message: micro pos
Parts:
- moved U1 300.3 mm to (25.5, 33.0), turned to -90 degrees
- moved D2 11.2 mm to (25.6, 52.5), turned to 180 degrees
- moved D1 2.66 mm to (36.0, 25.3)
- turned D48 to 90 degrees
Routing:
- net row0: track 0.00 -> 278.5 mm
- net row2: track 0.00 -> 275.6 mm
- net row3: track 0.00 -> 265.8 mm
- net Net-(D10-Pad1): track 0.00 -> 251.4 mm
- net Net-(D1-Pad2): track 0.00 -> 15.0 mm
- net Net-(D24-Pad2): track 0.00 -> 13.5 mm
- net Net-(D48-Pad2): track 0.00 -> 13.4 mm
- net Net-(D16-Pad2): track 0.00 -> 13.3 mm
- net Net-(D44-Pad2): track 0.00 -> 13.2 mm
- net Net-(D39-Pad2): track 0.00 -> 13.2 mm
- net Net-(D43-Pad2): track 0.00 -> 13.2 mm
- net Net-(D25-Pad2): track 0.00 -> 13.2 mm
- net Net-(D47-Pad2): track 0.00 -> 13.2 mm
- net Net-(D31-Pad2): track 0.00 -> 13.2 mm
- net Net-(D42-Pad2): track 0.00 -> 13.2 mm
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
Commit message: jefe final
Routing:
- net col14: track 0.00 -> 255.3 mm, vias 0 -> 1
- net col13: track 70.8 -> 296.0 mm, vias 0 -> 1
- net col12: track 67.0 -> 269.2 mm, vias 0 -> 1
- net col11: track 66.0 -> 249.0 mm, vias 0 -> 1
- net col10: track 44.0 -> 207.9 mm, vias 0 -> 1
- net col9: track 44.0 -> 188.8 mm, vias 0 -> 1
- net col8: track 44.0 -> 177.6 mm, vias 0 -> 1
- net col7: track 44.0 -> 159.6 mm, vias 0 -> 1
- net col6: track 44.0 -> 141.2 mm, vias 0 -> 1
- net col5: track 93.2 -> 172.1 mm, vias 0 -> 1
- net col4: track 72.1 -> 132.9 mm, vias 0 -> 1
- net col3: track 75.3 -> 117.8 mm, vias 0 -> 1
- net Net-(D10-Pad1): track 251.4 -> 277.2 mm
